Commit message: working with gazebo and state publisher urdf

File: models/capra6/capra6.urdf (robot description, URDF)
Before this commit: robot test_robot, 2 links, 1 joints
Links:
- removed link laser
- added link laser_link, mass 1; collision sphere radius=0.1; visual sphere radius=0.1
Joints:
- joint joint1: child laser -> laser_link

Commit message: changed link name to laser for compatibility with plugin

File: models/capra6/capra6.urdf (robot description, URDF)
Before this commit: robot capra6, 2 links, 1 joints
Links:
- removed link laser_link
- added link laser, mass 1; collision sphere radius=0.1; visual sphere radius=0.1
Joints:
- joint joint1: child laser_link -> laser
